File: PCBA/JouleCounter.kicad_sch (KiCad schematic)
At the start: 1 part, among them J101 JTAG

Commit message: Add Qwiic
Parts:
- added J102: Qwiic, Connector_JST:JST_SH_BM04B-SRSS-TB_1x04-1MP_P1.00mm_Vertical, symbol Connector_Generic_MountingPin:Conn_01x04_MountingPin
Connections:
- net GND: now also J102.1 (Pin_1), J102.MP (MountPin)
- net SCL: now also J102.4 (Pin_4)
- net SDA: now also J102.3 (Pin_3)
- net VDD: now also J102.2 (Pin_2)
Changed lines of the file:
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@@
   (junction (at 57.15 186.69) (diameter 0) (color 0 0 0 0)
+  )
+  (junction (at 266.7 158.75) (diameter 0) (color 0 0 0 0)
   )
   (polyline (pts (xy 228.6 12.7) (xy 228.6 166.37))
@@
     (stroke (width 0) (type default) (color 0 0 0 0))
   )
+  (wire (pts (xy 257.81 148.59) (xy 261.62 148.59))
+    (stroke (width 0) (type default) (color 0 0 0 0))
+  )
+  (wire (pts (xy 254 158.75) (xy 254 146.05))
+    (stroke (width 0) (type default) (color 0 0 0 0))
+  )
+  (wire (pts (xy 257.81 142.24) (xy 257.81 148.59))
+    (stroke (width 0) (type default) (color 0 0 0 0))
+  )
   (wire (pts (xy 57.15 181.61) (xy 57.15 184.15))
     (stroke (width 0) (type default) (color 0 0 0 0))
@@
     (stroke (width 0) (type default) (color 0 0 0 0))
   )
+  (wire (pts (xy 254 146.05) (xy 261.62 146.05))
+    (stroke (width 0) (type default) (color 0 0 0 0))
+  )
   (wire (pts (xy 57.15 186.69) (xy 57.15 189.23))
     (stroke (width 0) (type default) (color 0 0 0 0))
   )
   (wire (pts (xy 57.15 184.15) (xy 57.15 186.69))
+    (stroke (width 0) (type default) (color 0 0 0 0))
+  )
+  (wire (pts (xy 266.7 158.75) (xy 254 158.75))
     (stroke (width 0) (type default) (color 0 0 0 0))
   )
@@
     (effects (font (size 1.27 1.27)) (justify left bottom))
   )
-  (label "BootMode" (at 191.77 134.62 180)
+  (label "BootMode" (at 191.77 142.24 180)
     (effects (font (size 1.27 1.27)) (justify right bottom))
   )
@@
     (effects (font (size 1.27 1.27)) (justify left bottom))
   )
-  (label "Uart Tx" (at 101.6 106.68 0)
+  (label "Uart Tx" (at 76.2 83.82 0)
     (effects (font (size 1.27 1.27)) (justify left bottom))
   )
@@
     (effects (font (size 1.27 1.27)) (justify right bottom))
   )
-  (label "Button A" (at 191.77 137.16 180)
+  (label "Button A" (at 191.77 134.62 180)
+    (effects (font (size 1.27 1.27)) (justify right bottom))
+  )
+  (label "SDA" (at 261.62 151.13 180)
     (effects (font (size 1.27 1.27)) (justify right bottom))
   )
@@
     (effects (font (size 1.27 1.27)) (justify left bottom))
   )
-  (label "Uart Rx" (at 100.33 111.76 0)
+  (label "Uart Rx" (at 76.2 60.96 0)
     (effects (font (size 1.27 1.27)) (justify left bottom))
   )
@@
     (effects (font (size 1.27 1.27)) (justify right bottom))
   )
-  (label "Button B" (at 191.77 139.7 180)
+  (label "Button B" (at 191.77 137.16 180)
     (effects (font (size 1.27 1.27)) (justify right bottom))
   )
@@
     (effects (font (size 1.27 1.27)) (justify right bottom))
   )
-  (label "Button C" (at 191.77 142.24 180)
+  (label "Button C" (at 191.77 139.7 180)
     (effects (font (size 1.27 1.27)) (justify right bottom))
   )
@@
     (effects (font (size 1.27 1.27)) (justify left bottom))
   )
+  (label "SCL" (at 261.62 153.67 180)
+    (effects (font (size 1.27 1.27)) (justify right bottom))
+  )
   (label "Current ADC" (at 190.5 85.09 180)
     (effects (font (size 1.27 1.27)) (justify right bottom))
@@
   (label "USB D+ DAC{slash}ADC" (at 76.2 76.2 0)
     (effects (font (size 1.27 1.27)) (justify left bottom))
+  )
+  (symbol (lib_id "power:VDD") (at 257.81 142.24 0) (unit 1)
+    (in_bom yes) (on_board yes) (fields_autoplaced)
+    (property "Reference" "#PWR0121" (id 0) (at 257.81 146.05 0)
+      (effects (font (size 1.27 1.27)) hide)
+    )
+    (property "Value" "VDD" (id 1) (at 257.81 137.16 0))
+    (property "Footprint" "" (id 2) (at 257.81 142.24 0)
+      (effects (font (size 1.27 1.27)) hide)
+    )
+    (property "Datasheet" "" (id 3) (at 257.81 142.24 0)
+      (effects (font (size 1.27 1.27)) hide)
+    )
+    (pin "1")
   )
   (symbol (lib_id "Connector_Generic:Conn_02x05_Odd_Even") (at 62.23 184.15 0) (unit 1)
@@
     (pin "1")
   )
+  (symbol (lib_id "Connector_Generic_MountingPin:Conn_01x04_MountingPin") (at 266.7 148.59 0) (unit 1)
+    (in_bom yes) (on_board yes) (fields_autoplaced)
+    (property "Reference" "J102" (id 0) (at 269.24 148.9455 0)
+      (effects (font (size 1.27 1.27)) (justify left))
+    )
+    (property "Value" "Qwiic" (id 1) (at 269.24 151.4855 0)
+      (effects (font (size 1.27 1.27)) (justify left))
+    )
+    (property "Footprint" "Connector_JST:JST_SH_BM04B-SRSS-TB_1x04-1MP_P1.00mm_Vertical" (id 2) (at 266.7 148.59 0)
+      (effects (font (size 1.27 1.27)) hide)
+    )
+    (property "Datasheet" "~" (id 3) (at 266.7 148.59 0)
+      (effects (font (size 1.27 1.27)) hide)
+    )
+    (pin "1")
+    (pin "2")
+    (pin "3")
+    (pin "4")
+    (pin "MP")
+  )
+  (symbol (lib_id "power:GND") (at 266.7 158.75 0) (unit 1)
+    (in_bom yes) (on_board yes) (fields_autoplaced)
+    (property "Reference" "#PWR0120" (id 0) (at 266.7 165.1 0)
+      (effects (font (size 1.27 1.27)) hide)
+    )
+    (property "Value" "GND" (id 1) (at 266.7 163.83 0))
+    (property "Footprint" "" (id 2) (at 266.7 158.75 0)
+      (effects (font (size 1.27 1.27)) hide)
+    )
+    (property "Datasheet" "" (id 3) (at 266.7 158.75 0)
+      (effects (font (size 1.27 1.27)) hide)
+    )
+    (pin "1")
+  )
   (sheet (at 254 63.5) (size 25.4 25.4) (fields_autoplaced)
     (stroke (width 0.1524) (type solid) (color 0 0 0 0))
@@
       (reference "#PWR0119") (unit 1) (value "GND") (footprint "")
     )
+    (path "/e4f3ea4b-8548-461b-867e-ba5b81748be8"
+      (reference "#PWR0120") (unit 1) (value "GND") (footprint "")
+    )
+    (path "/3d172ed3-d962-432a-ab36-89a3c838f827"
+      (reference "#PWR0121") (unit 1) (value "VDD") (footprint "")
+    )
     (path "/7bd54514-8f0a-4683-8b19-da3af36c1bff/b00704da-7c99-4ac9-b795-5b97ca4da31f"
       (reference "#PWR0122") (unit 1) (value "GND") (footprint "")
@@
       (reference "#PWR0147") (unit 1) (value "VDD") (footprint "")
     )
+    (path "/61f092db-d732-44e6-ab5b-e56a273f9e01/885785e7-e551-43fa-9a0f-fe1eebaa3172"
+      (reference "#PWR0148") (unit 1) (value "VDD") (footprint "")
+    )
     (path "/61f092db-d732-44e6-ab5b-e56a273f9e01/76e48296-ced0-4a92-b314-8760d26ef2a9"
-      (reference "#PWR?") (unit 1) (value "GND") (footprint "")
-    )
-    (path "/61f092db-d732-44e6-ab5b-e56a273f9e01/885785e7-e551-43fa-9a0f-fe1eebaa3172"
-      (reference "#PWR?") (unit 1) (value "VDD") (footprint "")
+      (reference "#PWR0149") (unit 1) (value "GND") (footprint "")
+    )
+    (path "/61f092db-d732-44e6-ab5b-e56a273f9e01/e5f01fd5-d07e-4f17-bb11-d1cd1412c5e2"
+      (reference "#PWR0150") (unit 1) (value "GND") (footprint "")
     )
     (path "/61f092db-d732-44e6-ab5b-e56a273f9e01/9f678891-833a-4ca3-bcec-175ac5a6f206"
-      (reference "#PWR?") (unit 1) (value "GND") (footprint "")
-    )
-    (path "/61f092db-d732-44e6-ab5b-e56a273f9e01/e5f01fd5-d07e-4f17-bb11-d1cd1412c5e2"
-      (reference "#PWR?") (unit 1) (value "GND") (footprint "")
+      (reference "#PWR0151") (unit 1) (value "GND") (footprint "")
     )
     (path "/4847c8c0-6173-45c5-9b4b-8c9418cb5a91/5ab0d0b8-0dee-43b0-9b10-f6994da16df9"
@@
       (reference "J101") (unit 1) (value "JTAG") (footprint "")
     )
+    (path "/e3902119-c7f4-4332-a98e-a929c3b358a5"
+      (reference "J102") (unit 1) (value "Qwiic") (footprint "Connector_JST:JST_SH_BM04B-SRSS-TB_1x04-1MP_P1.00mm_Vertical")
+    )
     (path "/11e6ad7b-94c7-4abc-98e0-e4b10d097f65/849ef7e5-8097-4aee-8015-323905546838"
       (reference "J501") (unit 1) (value "USB_C_Receptacle") (footprint "Connector_USB:USB_C_Plug_JAE_DX07P024AJ1")
@@
     )
     (path "/61f092db-d732-44e6-ab5b-e56a273f9e01/3dcb82af-5522-4234-9097-cffd473db105"
-      (reference "Q?") (unit 1) (value "2N7002") (footprint "Package_TO_SOT_SMD:SOT-23")
+      (reference "Q701") (unit 1) (value "2N7002") (footprint "Package_TO_SOT_SMD:SOT-23")
     )
     (path "/4847c8c0-6173-45c5-9b4b-8c9418cb5a91/271287de-d1ab-46e7-9e8d-0eca17ee0aae"
@@
     )
     (path "/61f092db-d732-44e6-ab5b-e56a273f9e01/77068506-5e69-47f6-8c18-559ed07a8a9f"
-      (reference "R?") (unit 1) (value "200?") (footprint "")
+      (reference "R705") (unit 1) (value "200?") (footprint "")
     )
     (path "/61f092db-d732-44e6-ab5b-e56a273f9e01/d56e2cbb-18b1-4bbb-a667-68ae00ced67f"

Commit message: Start adding power
Other:
- added sheet Power (power.kicad_sch)
Changed lines of the file:
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@@
+    )
+  )
+  (sheet (at 127 127) (size 25.4 25.4) (fields_autoplaced)
+    (stroke (width 0.1524) (type solid) (color 0 0 0 0))
+    (fill (color 128 77 0 0.4000))
+    (property "Sheet name" "Power" (id 0) (at 127 126.2884 0)
+      (effects (font (size 1.27 1.27)) (justify left bottom))
+    )
+    (property "Sheet file" "power.kicad_sch" (id 1) (at 127 152.9846 0)
+      (effects (font (size 1.27 1.27)) (justify left top))
     )
   )
@@
     (path "/b0bcfef4-b206-452e-922a-e4174969def9" (page "6"))
     (path "/22f53838-7224-4d50-99f8-44746cd87af7" (page "7"))
+    (path "/3f787304-0f09-428f-9615-a178d53b5ed2" (page "8"))
     (path "/61f092db-d732-44e6-ab5b-e56a273f9e01" (page "8"))
   )
@@
       (reference "#PWR0151") (unit 1) (value "GND") (footprint "")
     )
+    (path "/3f787304-0f09-428f-9615-a178d53b5ed2/025baa4e-9c0e-4171-ba18-c81707277562"
+      (reference "#PWR?") (unit 1) (value "GND") (footprint "")
+    )
+    (path "/3f787304-0f09-428f-9615-a178d53b5ed2/ce52e298-4c1f-4e90-ab4b-157701b38695"
+      (reference "#PWR?") (unit 1) (value "VDD") (footprint "")
+    )
+    (path "/3f787304-0f09-428f-9615-a178d53b5ed2/e3b4b56e-1f52-450b-8489-ca84d306ba5d"
+      (reference "#PWR?") (unit 1) (value "GND") (footprint "")
+    )
     (path "/4847c8c0-6173-45c5-9b4b-8c9418cb5a91/5ab0d0b8-0dee-43b0-9b10-f6994da16df9"
       (reference "C201") (unit 1) (value "0.1uF") (footprint "Capacitor_SMD:C_0603_1608Metric")
@@
       (reference "C402") (unit 1) (value "1uF") (footprint "Capacitor_SMD:C_0603_1608Metric")
     )
+    (path "/3f787304-0f09-428f-9615-a178d53b5ed2/4eb5c59d-1379-4262-b562-de782e44eab1"
+      (reference "C?") (unit 1) (value "C") (footprint "")
+    )
+    (path "/3f787304-0f09-428f-9615-a178d53b5ed2/6ab14622-6f03-4c24-b5d4-28433b10dd40"
+      (reference "C?") (unit 1) (value "C") (footprint "")
+    )
+    (path "/3f787304-0f09-428f-9615-a178d53b5ed2/6fc95eb4-92c7-4d72-9433-c707bbf461a7"
+      (reference "C?") (unit 1) (value "C") (footprint "")
+    )
+    (path "/3f787304-0f09-428f-9615-a178d53b5ed2/8be65536-d759-4cf3-b037-dc944acc4618"
+      (reference "C?") (unit 1) (value "C") (footprint "")
+    )
+    (path "/3f787304-0f09-428f-9615-a178d53b5ed2/ab9857ff-be9c-4f4e-ac17-1db36b35c7f3"
+      (reference "C?") (unit 1) (value "C") (footprint "")
+    )
     (path "/83753f19-1938-4fce-8198-e7ca63503313"
       (reference "J101") (unit 1) (value "JTAG") (footprint "")
@@
       (reference "R705") (unit 1) (value "200?") (footprint "")
     )
+    (path "/3f787304-0f09-428f-9615-a178d53b5ed2/cb82b248-aec3-4ac6-aaea-dbb7ae20538e"
+      (reference "R?") (unit 1) (value "R") (footprint "")
+    )
     (path "/61f092db-d732-44e6-ab5b-e56a273f9e01/d56e2cbb-18b1-4bbb-a667-68ae00ced67f"
       (reference "SW801") (unit 1) (value "SW_Push") (footprint "Button_Switch_THT:SW_Tactile_SKHH_Angled")
@@
       (reference "U701") (unit 1) (value "INA181") (footprint "Package_TO_SOT_SMD:SOT-23-6")
     )
+    (path "/3f787304-0f09-428f-9615-a178d53b5ed2/1e50f7c6-3080-4467-aaf5-2bf00cdf949f"
+      (reference "U?") (unit 1) (value "TC2014-3.3VxCTTR") (footprint "Package_TO_SOT_SMD:SOT-23-5")
+    )
+    (path "/3f787304-0f09-428f-9615-a178d53b5ed2/2e20faf4-7401-46d5-ae6b-fc5bbb32f6ff"
+      (reference "U?") (unit 1) (value "LM5088-1") (footprint "Package_SO:HTSSOP-16-1EP_4.4x5mm_P0.65mm_EP3.4x5mm_Mask3x3mm_ThermalVias")
+    )
     (path "/4847c8c0-6173-45c5-9b4b-8c9418cb5a91/c5a59dc7-2bb1-40d5-9012-f726395f3506"

Commit message: GPIO association pass 1
Other:
- sheet Power ports: added 5V, VBus; removed none
Changed lines of the file:
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@@
     (effects (font (size 1.27 1.27)) (justify right bottom))
   )
-  (label "~{FUSB IRQ}" (at 100.33 53.34 0)
+  (label "~{FUSB IRQ}" (at 76.2 58.42 0)
     (effects (font (size 1.27 1.27)) (justify left bottom))
   )
@@
     (effects (font (size 1.27 1.27)) (justify right bottom))
   )
-  (label "SDA" (at 100.33 46.99 0)
+  (label "SDA" (at 76.2 66.04 0)
     (effects (font (size 1.27 1.27)) (justify left bottom))
   )
@@
     (effects (font (size 1.27 1.27)) (justify left bottom))
   )
-  (label "JTAG TCK" (at 101.6 81.28 0)
-    (effects (font (size 1.27 1.27)) (justify left bottom))
-  )
-  (label "LCD COPI" (at 101.6 92.71 0)
+  (label "JTAG TCK" (at 76.2 48.26 0)
+    (effects (font (size 1.27 1.27)) (justify left bottom))
+  )
+  (label "LCD COPI" (at 76.2 86.36 0)
     (effects (font (size 1.27 1.27)) (justify left bottom))
   )
@@
     (effects (font (size 1.27 1.27)) (justify left bottom))
   )
+  (label "5V_USB" (at 152.4 130.81 0)
+    (effects (font (size 1.27 1.27)) (justify left bottom))
+  )
   (label "JTAG TDO" (at 69.85 184.15 0)
     (effects (font (size 1.27 1.27)) (justify left bottom))
@@
     (effects (font (size 1.27 1.27)) (justify left bottom))
   )
-  (label "LCD SCK" (at 101.6 90.17 0)
-    (effects (font (size 1.27 1.27)) (justify left bottom))
-  )
-  (label "VBus ADC" (at 100.33 66.04 0)
+  (label "LCD SCK" (at 76.2 91.44 0)
+    (effects (font (size 1.27 1.27)) (justify left bottom))
+  )
+  (label "VBus" (at 152.4 137.16 0)
+    (effects (font (size 1.27 1.27)) (justify left bottom))
+  )
+  (label "VBus ADC" (at 76.2 53.34 0)
     (effects (font (size 1.27 1.27)) (justify left bottom))
   )
@@
     (effects (font (size 1.27 1.27)) (justify left bottom))
   )
-  (label "JTAG TDI" (at 101.6 83.82 0)
+  (label "JTAG TDI" (at 76.2 45.72 0)
     (effects (font (size 1.27 1.27)) (justify left bottom))
   )
@@
     (effects (font (size 1.27 1.27)) (justify right bottom))
   )
-  (label "LCD CS" (at 101.6 97.79 0)
+  (label "LCD CS" (at 76.2 88.9 0)
     (effects (font (size 1.27 1.27)) (justify left bottom))
   )
@@
     (effects (font (size 1.27 1.27)) (justify left bottom))
   )
+  (label "5V_USB" (at 254 105.41 180)
+    (effects (font (size 1.27 1.27)) (justify right bottom))
+  )
   (label "~{FUSB IRQ}" (at 190.5 58.42 180)
     (effects (font (size 1.27 1.27)) (justify right bottom))
   )
-  (label "LCD PWM" (at 101.6 100.33 0)
+  (label "LCD PWM" (at 76.2 71.12 0)
     (effects (font (size 1.27 1.27)) (justify left bottom))
   )
@@
     (effects (font (size 1.27 1.27)) (justify left bottom))
   )
-  (label "JTAG TMS" (at 101.6 86.36 0)
+  (label "JTAG TMS" (at 76.2 43.18 0)
     (effects (font (size 1.27 1.27)) (justify left bottom))
   )
@@
     (effects (font (size 1.27 1.27)) (justify right bottom))
   )
-  (label "LCD DC" (at 101.6 95.25 0)
+  (label "LCD DC" (at 76.2 73.66 0)
     (effects (font (size 1.27 1.27)) (justify left bottom))
   )
@@
     (effects (font (size 1.27 1.27)) (justify left bottom))
   )
-  (label "Current ADC" (at 100.33 68.58 0)
+  (label "Current ADC" (at 76.2 55.88 0)
     (effects (font (size 1.27 1.27)) (justify left bottom))
   )
@@
     (effects (font (size 1.27 1.27)) (justify right bottom))
   )
-  (label "SCL" (at 100.33 49.53 0)
+  (label "SCL" (at 76.2 68.58 0)
     (effects (font (size 1.27 1.27)) (justify left bottom))
   )
@@
     (effects (font (size 1.27 1.27)) (justify right bottom))
   )
-  (label "JTAG TDO" (at 101.6 78.74 0)
+  (label "JTAG TDO" (at 76.2 50.8 0)
     (effects (font (size 1.27 1.27)) (justify left bottom))
   )
@@
       (effects (font (size 1.27 1.27)) (justify left top))
     )
-  )
+    (pin "5V" input (at 152.4 130.81 0)
+      (effects (font (size 1.27 1.27)) (justify right))
+    )
+    (pin "VBus" input (at 152.4 137.16 0)
+      (effects (font (size 1.27 1.27)) (justify right))
+    )
+  )

Commit message: Assign footprints
Parts:
- J101: footprint (none) -> Connector_PinHeader_2.54mm:PinHeader_2x05_P2.54mm_Vertical
