File: PCBA/JouleCounter.kicad_sch (KiCad schematic)
At the start: 0 parts

Commit message: Finish routing
Parts:
- added R101: 10k, Resistor_SMD:R_0603_1608Metric, symbol Device:R
Connections:
- new net UI/~{LCD Reset}: R101.1
- new net VDD: R101.2
Changed lines of the file:
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@@
+    (stroke (width 0) (type default) (color 0 0 0 0))
+  )
+  (wire (pts (xy 215.9 134.62) (xy 219.71 134.62))
     (stroke (width 0) (type default) (color 0 0 0 0))
   )
@@
     (effects (font (size 1.27 1.27)) (justify left bottom))
   )
-  (label "~{Reset}" (at 215.9 134.62 0)
-    (effects (font (size 1.27 1.27)) (justify left bottom))
-  )
   (label "Uart Rx" (at 254 116.84 180)
     (effects (font (size 1.27 1.27)) (justify right bottom))
@@
   (label "Button A" (at 76.2 111.76 0)
     (effects (font (size 1.27 1.27)) (justify left bottom))
+  )
+  (symbol (lib_id "Device:R") (at 219.71 130.81 180) (unit 1)
+    (in_bom yes) (on_board yes)
+    (property "Reference" "R101" (id 0) (at 222.25 130.81 90))
+    (property "Value" "10k" (id 1) (at 219.71 130.81 90))
+    (property "Footprint" "Resistor_SMD:R_0603_1608Metric" (id 2) (at 221.488 130.81 90)
+      (effects (font (size 1.27 1.27)) hide)
+    )
+    (property "Datasheet" "~" (id 3) (at 219.71 130.81 0)
+      (effects (font (size 1.27 1.27)) hide)
+    )
+    (pin "1")
+    (pin "2")
+  )
+  (symbol (lib_id "power:VDD") (at 219.71 127 0) (unit 1)
+    (in_bom yes) (on_board yes) (fields_autoplaced)
+    (property "Reference" "#PWR0127" (id 0) (at 219.71 130.81 0)
+      (effects (font (size 1.27 1.27)) hide)
+    )
+    (property "Value" "VDD" (id 1) (at 219.71 121.92 0))
+    (property "Footprint" "" (id 2) (at 219.71 127 0)
+      (effects (font (size 1.27 1.27)) hide)
+    )
+    (property "Datasheet" "" (id 3) (at 219.71 127 0)
+      (effects (font (size 1.27 1.27)) hide)
+    )
+    (pin "1")
   )
   (sheet (at 254 63.5) (size 25.4 25.4) (fields_autoplaced)
@@
       (reference "#PWR0126") (unit 1) (value "VDD") (footprint "")
     )
+    (path "/c981e8fc-c1c6-4626-895f-d7ba18f4a276"
+      (reference "#PWR0127") (unit 1) (value "VDD") (footprint "")
+    )
+    (path "/61f092db-d732-44e6-ab5b-e56a273f9e01/c9c06e7a-c755-4710-bdb5-e2ed07d62edd"
+      (reference "#PWR0128") (unit 1) (value "GND") (footprint "")
+    )
     (path "/4847c8c0-6173-45c5-9b4b-8c9418cb5a91/6504199d-45c4-49cf-9a58-0af0267b5b71"
       (reference "#PWR0129") (unit 1) (value "GND") (footprint "")
@@
       (reference "Q701") (unit 1) (value "2N7002") (footprint "Package_TO_SOT_SMD:SOT-23")
     )
+    (path "/462d169a-9ddd-46c3-b556-917180b3c53d"
+      (reference "R101") (unit 1) (value "10k") (footprint "Resistor_SMD:R_0603_1608Metric")
+    )
     (path "/4847c8c0-6173-45c5-9b4b-8c9418cb5a91/271287de-d1ab-46e7-9e8d-0eca17ee0aae"
