File: PCBA/adc.kicad_sch (KiCad schematic)
At the start: 5 parts

Commit message: More schematics
Parts:
- R701, R702, R703, R704: renamed from R?; footprint (none) -> Resistor_SMD:R_0603_1608Metric
- gave numbers to parts that had none: 1
Changed lines of the file:
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@@
   (symbol (lib_id "power:GND") (at 114.3 93.98 0) (unit 1)
     (in_bom yes) (on_board yes) (fields_autoplaced)
-    (property "Reference" "#PWR?" (id 0) (at 114.3 100.33 0)
+    (property "Reference" "#PWR0143" (id 0) (at 114.3 100.33 0)
       (effects (font (size 1.27 1.27)) hide)
     )
@@
   (symbol (lib_id "power:VDD") (at 114.3 76.2 0) (unit 1)
     (in_bom yes) (on_board yes) (fields_autoplaced)
-    (property "Reference" "#PWR?" (id 0) (at 114.3 80.01 0)
+    (property "Reference" "#PWR0140" (id 0) (at 114.3 80.01 0)
       (effects (font (size 1.27 1.27)) hide)
     )
@@
   (symbol (lib_id "Device:R") (at 88.9 90.17 0) (unit 1)
     (in_bom yes) (on_board yes) (fields_autoplaced)
-    (property "Reference" "R?" (id 0) (at 91.44 88.8999 0)
+    (property "Reference" "R702" (id 0) (at 91.44 88.8999 0)
       (effects (font (size 1.27 1.27)) (justify left))
     )
@@
       (effects (font (size 1.27 1.27)) (justify left))
     )
-    (property "Footprint" "" (id 2) (at 87.122 90.17 90)
+    (property "Footprint" "Resistor_SMD:R_0603_1608Metric" (id 2) (at 87.122 90.17 90)
       (effects (font (size 1.27 1.27)) hide)
     )
@@
   (symbol (lib_id "Device:R") (at 114.3 90.17 0) (unit 1)
     (in_bom yes) (on_board yes) (fields_autoplaced)
-    (property "Reference" "R?" (id 0) (at 116.84 88.8999 0)
+    (property "Reference" "R704" (id 0) (at 116.84 88.8999 0)
       (effects (font (size 1.27 1.27)) (justify left))
     )
@@
       (effects (font (size 1.27 1.27)) (justify left))
     )
-    (property "Footprint" "" (id 2) (at 112.522 90.17 90)
+    (property "Footprint" "Resistor_SMD:R_0603_1608Metric" (id 2) (at 112.522 90.17 90)
       (effects (font (size 1.27 1.27)) hide)
     )
@@
   (symbol (lib_id "power:GND") (at 152.4 90.17 0) (unit 1)
     (in_bom yes) (on_board yes) (fields_autoplaced)
-    (property "Reference" "#PWR?" (id 0) (at 152.4 96.52 0)
+    (property "Reference" "#PWR0141" (id 0) (at 152.4 96.52 0)
       (effects (font (size 1.27 1.27)) hide)
     )
@@
   (symbol (lib_id "power:GND") (at 88.9 93.98 0) (unit 1)
     (in_bom yes) (on_board yes) (fields_autoplaced)
-    (property "Reference" "#PWR?" (id 0) (at 88.9 100.33 0)
+    (property "Reference" "#PWR0139" (id 0) (at 88.9 100.33 0)
       (effects (font (size 1.27 1.27)) hide)
     )
@@
   (symbol (lib_id "power:VDD") (at 152.4 74.93 0) (unit 1)
     (in_bom yes) (on_board yes) (fields_autoplaced)
-    (property "Reference" "#PWR?" (id 0) (at 152.4 78.74 0)
+    (property "Reference" "#PWR0142" (id 0) (at 152.4 78.74 0)
       (effects (font (size 1.27 1.27)) hide)
     )
@@
   (symbol (lib_id "Device:R") (at 114.3 80.01 0) (unit 1)
     (in_bom yes) (on_board yes) (fields_autoplaced)
-    (property "Reference" "R?" (id 0) (at 116.84 78.7399 0)
+    (property "Reference" "R703" (id 0) (at 116.84 78.7399 0)
       (effects (font (size 1.27 1.27)) (justify left))
     )
@@
       (effects (font (size 1.27 1.27)) (justify left))
     )
-    (property "Footprint" "" (id 2) (at 112.522 80.01 90)
+    (property "Footprint" "Resistor_SMD:R_0603_1608Metric" (id 2) (at 112.522 80.01 90)
       (effects (font (size 1.27 1.27)) hide)
     )
@@
   (symbol (lib_id "Amplifier_Current:INA181") (at 154.94 82.55 0) (unit 1)
     (in_bom yes) (on_board yes) (fields_autoplaced)
-    (property "Reference" "U?" (id 0) (at 165.1 77.851 0))
+    (property "Reference" "U701" (id 0) (at 165.1 77.851 0))
     (property "Value" "INA181" (id 1) (at 165.1 80.391 0))
     (property "Footprint" "Package_TO_SOT_SMD:SOT-23-6" (id 2) (at 156.21 81.28 0)
@@
   (symbol (lib_id "Device:R") (at 88.9 80.01 0) (unit 1)
     (in_bom yes) (on_board yes) (fields_autoplaced)
-    (property "Reference" "R?" (id 0) (at 91.44 78.7399 0)
+    (property "Reference" "R701" (id 0) (at 91.44 78.7399 0)
       (effects (font (size 1.27 1.27)) (justify left))
     )
@@
       (effects (font (size 1.27 1.27)) (justify left))
     )
-    (property "Footprint" "" (id 2) (at 87.122 80.01 90)
+    (property "Footprint" "Resistor_SMD:R_0603_1608Metric" (id 2) (at 87.122 80.01 90)
       (effects (font (size 1.27 1.27)) hide)
     )

Commit message: molex model
Parts:
- removed R701: 1.4M, Resistor_SMD:R_0603_1608Metric, symbol Device:R
- removed R702, R703, R704: 100K, Resistor_SMD:R_0603_1608Metric, symbol Device:R
- removed U701: INA181, Package_TO_SOT_SMD:SOT-23-6, symbol Amplifier_Current:INA181
- added U701: INA226, Package_SO:VSSOP-10_3x3mm_P0.5mm, symbol Analog_ADC:INA226
Connections:
- net GND: now also U701.1 (A1), U701.2 (A0), U701.7 (GND)
- net VDD: now also U701.6 (VS)
- new net SCL: U701.5 (SCL)
- new net SDA: U701.4 (SDA)
- new net Vsense+: U701.10 (Vin+), U701.8 (Vbus)
- new net Vsense-: U701.9 (Vin-)
- new net ~{ALERT}: U701.3 (~{Alert})
Other:
- note removed: "INA181A1IDBVR In stock at LCSC A1 is 20x gain Therefore want 0.165V at 5+A 0.02 ohm shunt gets us close"
Changed lines of the file:
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@@
 (kicad_sch (version 20211123) (generator eeschema)
   (paper "A4")
-  (junction (at 114.3 85.09) (diameter 0) (color 0 0 0 0)
+  (junction (at 177.8 101.6) (diameter 0) (color 0 0 0 0)
   )
-  (junction (at 88.9 85.09) (diameter 0) (color 0 0 0 0)
+  (junction (at 177.8 80.01) (diameter 0) (color 0 0 0 0)
   )
-  (wire (pts (xy 93.98 85.09) (xy 88.9 85.09))
+  (wire (pts (xy 177.8 77.47) (xy 177.8 80.01))
     (stroke (width 0) (type default) (color 0 0 0 0))
   )
-  (wire (pts (xy 114.3 85.09) (xy 114.3 83.82))
+  (wire (pts (xy 153.67 80.01) (xy 177.8 80.01))
     (stroke (width 0) (type default) (color 0 0 0 0))
   )
-  (wire (pts (xy 88.9 85.09) (xy 88.9 83.82))
+  (wire (pts (xy 177.8 80.01) (xy 177.8 101.6))
     (stroke (width 0) (type default) (color 0 0 0 0))
   )
-  (wire (pts (xy 88.9 85.09) (xy 88.9 86.36))
+  (wire (pts (xy 143.51 101.6) (xy 143.51 97.79))
     (stroke (width 0) (type default) (color 0 0 0 0))
   )
-  (wire (pts (xy 114.3 85.09) (xy 114.3 86.36))
+  (wire (pts (xy 177.8 101.6) (xy 143.51 101.6))
     (stroke (width 0) (type default) (color 0 0 0 0))
   )
-  (wire (pts (xy 119.38 85.09) (xy 114.3 85.09))
+  (wire (pts (xy 153.67 77.47) (xy 177.8 77.47))
     (stroke (width 0) (type default) (color 0 0 0 0))
   )
-  (text "INA181A1IDBVR\nIn stock at LCSC\nA1 is 20x gain\nTherefore want 0.165V at 5+A\n0.02 ohm shunt gets us close"
-    (at 168.91 97.79 0)
-    (effects (font (size 1.27 1.27)) (justify left bottom))
-  )
-  (label "VRef" (at 157.48 90.17 0)
-    (effects (font (size 1.27 1.27)) (justify left bottom))
-  )
-  (label "VRef" (at 119.38 85.09 0)
-    (effects (font (size 1.27 1.27)) (justify left bottom))
-  )
-  (hierarchical_label "VBus In" (shape input) (at 88.9 76.2 0)
+  (hierarchical_label "SDA" (shape input) (at 153.67 85.09 0)
     (effects (font (size 1.27 1.27)) (justify left))
   )
-  (hierarchical_label "I Sense 2" (shape input) (at 147.32 85.09 180)
+  (hierarchical_label "Vsense-" (shape input) (at 133.35 90.17 180)
     (effects (font (size 1.27 1.27)) (justify right))
   )
-  (hierarchical_label "ADC VBus" (shape input) (at 93.98 85.09 0)
+  (hierarchical_label "Vsense+" (shape input) (at 133.35 87.63 180)
+    (effects (font (size 1.27 1.27)) (justify right))
+  )
+  (hierarchical_label "~{ALERT}" (shape input) (at 153.67 92.71 0)
     (effects (font (size 1.27 1.27)) (justify left))
   )
-  (hierarchical_label "I Sense 1" (shape input) (at 147.32 80.01 180)
+  (hierarchical_label "Vsense+" (shape input) (at 133.35 77.47 180)
     (effects (font (size 1.27 1.27)) (justify right))
   )
-  (hierarchical_label "ADC Current" (shape input) (at 162.56 82.55 0)
+  (hierarchical_label "SCL" (shape input) (at 153.67 87.63 0)
     (effects (font (size 1.27 1.27)) (justify left))
   )
-  (symbol (lib_id "power:GND") (at 114.3 93.98 0) (unit 1)
+  (symbol (lib_id "power:GND") (at 177.8 101.6 0) (unit 1)
     (in_bom yes) (on_board yes) (fields_autoplaced)
-    (property "Reference" "#PWR0143" (id 0) (at 114.3 100.33 0)
+    (property "Reference" "#PWR0135" (id 0) (at 177.8 107.95 0)
       (effects (font (size 1.27 1.27)) hide)
     )
-    (property "Value" "GND" (id 1) (at 114.3 99.06 0))
-    (property "Footprint" "" (id 2) (at 114.3 93.98 0)
+    (property "Value" "GND" (id 1) (at 177.8 106.68 0))
+    (property "Footprint" "" (id 2) (at 177.8 101.6 0)
       (effects (font (size 1.27 1.27)) hide)
     )
-    (property "Datasheet" "" (id 3) (at 114.3 93.98 0)
+    (property "Datasheet" "" (id 3) (at 177.8 101.6 0)
       (effects (font (size 1.27 1.27)) hide)
     )
     (pin "1")
   )
-  (symbol (lib_id "power:VDD") (at 114.3 76.2 0) (unit 1)
+  (symbol (lib_id "power:VDD") (at 143.51 72.39 0) (unit 1)
     (in_bom yes) (on_board yes) (fields_autoplaced)
-    (property "Reference" "#PWR0140" (id 0) (at 114.3 80.01 0)
+    (property "Reference" "#PWR0134" (id 0) (at 143.51 76.2 0)
       (effects (font (size 1.27 1.27)) hide)
     )
-    (property "Value" "VDD" (id 1) (at 114.3 71.12 0))
-    (property "Footprint" "" (id 2) (at 114.3 76.2 0)
+    (property "Value" "VDD" (id 1) (at 143.51 67.31 0))
+    (property "Footprint" "" (id 2) (at 143.51 72.39 0)
       (effects (font (size 1.27 1.27)) hide)
     )
-    (property "Datasheet" "" (id 3) (at 114.3 76.2 0)
+    (property "Datasheet" "" (id 3) (at 143.51 72.39 0)
       (effects (font (size 1.27 1.27)) hide)
     )
     (pin "1")
   )
-  (symbol (lib_id "Device:R") (at 88.9 90.17 0) (unit 1)
+  (symbol (lib_id "Analog_ADC:INA226") (at 143.51 85.09 0) (unit 1)
     (in_bom yes) (on_board yes) (fields_autoplaced)
-    (property "Reference" "R702" (id 0) (at 91.44 88.8999 0)
+    (property "Reference" "U701" (id 0) (at 145.5294 69.85 0)
       (effects (font (size 1.27 1.27)) (justify left))
     )
-    (property "Value" "100K" (id 1) (at 91.44 91.4399 0)
+    (property "Value" "INA226" (id 1) (at 145.5294 72.39 0)
       (effects (font (size 1.27 1.27)) (justify left))
     )
-    (property "Footprint" "Resistor_SMD:R_0603_1608Metric" (id 2) (at 87.122 90.17 90)
+    (property "Footprint" "Package_SO:VSSOP-10_3x3mm_P0.5mm" (id 2) (at 163.83 96.52 0)
       (effects (font (size 1.27 1.27)) hide)
     )
-    (property "Datasheet" "~" (id 3) (at 88.9 90.17 0)
+    (property "Datasheet" "http://www.ti.com/lit/ds/symlink/ina226.pdf" (id 3) (at 152.4 87.63 0)
       (effects (font (size 1.27 1.27)) hide)
     )
     (pin "1")
-    (pin "2")
-  )
-  (symbol (lib_id "Device:R") (at 114.3 90.17 0) (unit 1)
-    (in_bom yes) (on_board yes) (fields_autoplaced)
-    (property "Reference" "R704" (id 0) (at 116.84 88.8999 0)
-      (effects (font (size 1.27 1.27)) (justify left))
-    )
-    (property "Value" "100K" (id 1) (at 116.84 91.4399 0)
-      (effects (font (size 1.27 1.27)) (justify left))
-    )
-    (property "Footprint" "Resistor_SMD:R_0603_1608Metric" (id 2) (at 112.522 90.17 90)
-      (effects (font (size 1.27 1.27)) hide)
-    )
-    (property "Datasheet" "~" (id 3) (at 114.3 90.17 0)
-      (effects (font (size 1.27 1.27)) hide)
-    )
-    (pin "1")
-    (pin "2")
-  )
-  (symbol (lib_id "power:GND") (at 152.4 90.17 0) (unit 1)
-    (in_bom yes) (on_board yes) (fields_autoplaced)
-    (property "Reference" "#PWR0141" (id 0) (at 152.4 96.52 0)
-      (effects (font (size 1.27 1.27)) hide)
-    )
-    (property "Value" "GND" (id 1) (at 152.4 95.25 0))
-    (property "Footprint" "" (id 2) (at 152.4 90.17 0)
-      (effects (font (size 1.27 1.27)) hide)
-    )
-    (property "Datasheet" "" (id 3) (at 152.4 90.17 0)
-      (effects (font (size 1.27 1.27)) hide)
-    )
-    (pin "1")
-  )
-  (symbol (lib_id "power:GND") (at 88.9 93.98 0) (unit 1)
-    (in_bom yes) (on_board yes) (fields_autoplaced)
-    (property "Reference" "#PWR0139" (id 0) (at 88.9 100.33 0)
-      (effects (font (size 1.27 1.27)) hide)
-    )
-    (property "Value" "GND" (id 1) (at 88.9 99.06 0))
-    (property "Footprint" "" (id 2) (at 88.9 93.98 0)
-      (effects (font (size 1.27 1.27)) hide)
-    )
-    (property "Datasheet" "" (id 3) (at 88.9 93.98 0)
-      (effects (font (size 1.27 1.27)) hide)
-    )
-    (pin "1")
-  )
-  (symbol (lib_id "power:VDD") (at 152.4 74.93 0) (unit 1)
-    (in_bom yes) (on_board yes) (fields_autoplaced)
-    (property "Reference" "#PWR0142" (id 0) (at 152.4 78.74 0)
-      (effects (font (size 1.27 1.27)) hide)
-    )
-    (property "Value" "VDD" (id 1) (at 152.4 69.85 0))
-    (property "Footprint" "" (id 2) (at 152.4 74.93 0)
-      (effects (font (size 1.27 1.27)) hide)
-    )
-    (property "Datasheet" "" (id 3) (at 152.4 74.93 0)
-      (effects (font (size 1.27 1.27)) hide)
-    )
-    (pin "1")
-  )
-  (symbol (lib_id "Device:R") (at 114.3 80.01 0) (unit 1)
-    (in_bom yes) (on_board yes) (fields_autoplaced)
-    (property "Reference" "R703" (id 0) (at 116.84 78.7399 0)
-      (effects (font (size 1.27 1.27)) (justify left))
-    )
-    (property "Value" "100K" (id 1) (at 116.84 81.2799 0)
-      (effects (font (size 1.27 1.27)) (justify left))
-    )
-    (property "Footprint" "Resistor_SMD:R_0603_1608Metric" (id 2) (at 112.522 80.01 90)
-      (effects (font (size 1.27 1.27)) hide)
-    )
-    (property "Datasheet" "~" (id 3) (at 114.3 80.01 0)
-      (effects (font (size 1.27 1.27)) hide)
-    )
-    (pin "1")
-    (pin "2")
-  )
-  (symbol (lib_id "Amplifier_Current:INA181") (at 154.94 82.55 0) (unit 1)
-    (in_bom yes) (on_board yes) (fields_autoplaced)
-    (property "Reference" "U701" (id 0) (at 165.1 77.851 0))
-    (property "Value" "INA181" (id 1) (at 165.1 80.391 0))
-    (property "Footprint" "Package_TO_SOT_SMD:SOT-23-6" (id 2) (at 156.21 81.28 0)
-      (effects (font (size 1.27 1.27)) hide)
-    )
-    (property "Datasheet" "http://www.ti.com/lit/ds/symlink/ina181.pdf" (id 3) (at 158.75 78.74 0)
-      (effects (font (size 1.27 1.27)) hide)
-    )
-    (pin "1")
+    (pin "10")
     (pin "2")
     (pin "3")
@@
     (pin "5")
     (pin "6")
-  )
-  (symbol (lib_id "Device:R") (at 88.9 80.01 0) (unit 1)
-    (in_bom yes) (on_board yes) (fields_autoplaced)
-    (property "Reference" "R701" (id 0) (at 91.44 78.7399 0)
-      (effects (font (size 1.27 1.27)) (justify left))
-    )
-    (property "Value" "1.4M" (id 1) (at 91.44 81.2799 0)
-      (effects (font (size 1.27 1.27)) (justify left))
-    )
-    (property "Footprint" "Resistor_SMD:R_0603_1608Metric" (id 2) (at 87.122 80.01 90)
-      (effects (font (size 1.27 1.27)) hide)
-    )
-    (property "Datasheet" "~" (id 3) (at 88.9 80.01 0)
-      (effects (font (size 1.27 1.27)) hide)
-    )
-    (pin "1")
-    (pin "2")
+    (pin "7")
+    (pin "8")
+    (pin "9")
   )
 )
