File: PCBA/ui.kicad_sch (KiCad schematic)
At the start: 14 parts, among them J901 Conn_02x25_Odd_Even_MountingP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, Q701 2N7002, SW801 SW_Push, SW802 SW_Push, SW803 SW_Push, U901 LP2985-2.8

Commit message: molex model
Parts:
- removed C907: C, Capacitor_SMD:C_0603_1608Metric, symbol Device:C
Changed lines of the file:
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@@
   (junction (at 254 91.44) (diameter 0) (color 0 0 0 0)
-  )
-  (junction (at 182.88 158.75) (diameter 0) (color 0 0 0 0)
   )
   (junction (at 241.3 127) (diameter 0) (color 0 0 0 0)
@@
     (stroke (width 0) (type default) (color 0 0 0 0))
   )
-  (wire (pts (xy 182.88 158.75) (xy 198.12 158.75))
+  (wire (pts (xy 172.72 158.75) (xy 198.12 158.75))
     (stroke (width 0) (type default) (color 0 0 0 0))
   )
@@
   )
   (wire (pts (xy 182.88 101.6) (xy 182.88 66.04))
-    (stroke (width 0) (type default) (color 0 0 0 0))
-  )
-  (wire (pts (xy 172.72 158.75) (xy 182.88 158.75))
     (stroke (width 0) (type default) (color 0 0 0 0))
   )
@@
     (pin "3")
   )
-  (symbol (lib_id "Device:C") (at 182.88 154.94 0) (unit 1)
-    (in_bom yes) (on_board yes) (fields_autoplaced)
-    (property "Reference" "C907" (id 0) (at 186.69 153.6699 0)
-      (effects (font (size 1.27 1.27)) (justify left))
-    )
-    (property "Value" "C" (id 1) (at 186.69 156.2099 0)
-      (effects (font (size 1.27 1.27)) (justify left))
-    )
-    (property "Footprint" "Capacitor_SMD:C_0603_1608Metric" (id 2) (at 183.8452 158.75 0)
-      (effects (font (size 1.27 1.27)) hide)
-    )
-    (property "Datasheet" "~" (id 3) (at 182.88 154.94 0)
-      (effects (font (size 1.27 1.27)) hide)
-    )
-    (pin "1")
-    (pin "2")
-  )
   (symbol (lib_id "Device:C") (at 213.36 154.94 0) (unit 1)

Commit message: Finish routing
Connections:
- net GND: now also J901.MP (MountPin)
Changed lines of the file:
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@@
   (no_connect (at 224.79 71.12))
   (no_connect (at 224.79 73.66))
+  (wire (pts (xy 203.2 52.07) (xy 218.44 52.07))
+    (stroke (width 0) (type default) (color 0 0 0 0))
+  )
   (wire (pts (xy 190.5 81.28) (xy 212.09 81.28))
     (stroke (width 0) (type default) (color 0 0 0 0))
@@
   )
   (wire (pts (xy 254 96.52) (xy 254 116.84))
+    (stroke (width 0) (type default) (color 0 0 0 0))
+  )
+  (wire (pts (xy 218.44 52.07) (xy 218.44 53.34))
     (stroke (width 0) (type default) (color 0 0 0 0))
   )
@@
       (effects (font (size 1.27 1.27)) hide)
     )
+    (pin "1")
+  )
+  (symbol (lib_id "power:GND") (at 203.2 52.07 0) (unit 1)
+    (in_bom yes) (on_board yes) (fields_autoplaced)
+    (property "Reference" "#PWR0128" (id 0) (at 203.2 58.42 0)
+      (effects (font (size 1.27 1.27)) hide)
+    )
+    (property "Value" "GND" (id 1) (at 203.2 57.15 0))
+    (property "Footprint" "" (id 2) (at 203.2 52.07 0)
+      (effects (font (size 1.27 1.27)) hide)
+    )
+    (property "Datasheet" "" (id 3) (at 203.2 52.07 0)
+      (effects (font (size 1.27 1.27)) hide)
+    )
